Commit message: Latest update

File: iris_coastline/worlds/iris_coastline.world.xacro (robot description, xacro)
@@ -7,5 +7,5 @@
     <!--Waves-->
     <xacro:include filename="$(find wave_gazebo)/world_models/ocean_waves/model.xacro"/>
-    <xacro:ocean_waves/>
+    <xacro:ocean_waves gain="0.8" period="10"/>
     <!-- <include>
       <uri>model://robotx_navigation_challenge</uri>

File: vrx/wave_gazebo/world_models/ocean_waves/model.xacro (robot description, xacro)
@@ -17,7 +17,7 @@
 -->
 <world xmlns:xacro="http://ros.org/wiki/xacro">
-  <xacro:macro name="ocean_waves" params="gain:=0.1 period:=5
+  <xacro:macro name="ocean_waves" params="gain:=1.0 period:=5
                      direction_x:=1.0 direction_y:=0.0
-                     angle:=0.4 scale:=1.5">
+                     angle:=0.4 scale:=1.06">
   <model name='ocean_waves'>
     <static>true</static>

Commit message: Re-organize the file system of the current branch

File: iris_coastline/worlds/iris_coastline.world.xacro (robot description, xacro)
@@ -7,5 +7,5 @@
     <!--Waves-->
     <xacro:include filename="$(find wave_gazebo)/world_models/ocean_waves/model.xacro"/>
-    <xacro:ocean_waves gain="0.8" period="10"/>
+    <xacro:ocean_waves/>
     <!-- <include>
       <uri>model://robotx_navigation_challenge</uri>

File: vrx/wave_gazebo/world_models/ocean_waves/model.xacro (robot description, xacro)
@@ -17,7 +17,7 @@
 -->
 <world xmlns:xacro="http://ros.org/wiki/xacro">
-  <xacro:macro name="ocean_waves" params="gain:=1.0 period:=5
+  <xacro:macro name="ocean_waves" params="gain:=1.2 period:=5
                      direction_x:=1.0 direction_y:=0.0
-                     angle:=0.4 scale:=1.06">
+                     angle:=0.4 scale:=1.4">
   <model name='ocean_waves'>
     <static>true</static>
